File: hardware-pcb/JukeBox.kicad_sch (KiCad schematic)
At the start: 101 parts, among them J1 USB_C_Receptacle_USB2.0_16P, Q1 Q_NPN_BEC, SW1 SW_SPST, SW10 SW_SPST, SW11 SW_SPST, SW12 SW_SPST, SW2 SW_SPST, SW3 SW_SPST, SW4 SW_SPST, SW5 SW_SPST, SW6 SW_SPST, SW7 SW_SPST, SW8 SW_SPST, SW9 SW_SPST, U1 NCP1117-3.3_SOT223, U2 W25Q128JVS, U3 RP2040, U4 st7789v, U5 CAT24C512, Y2 ABM8-272-T3

Commit message: switch certain caps back to 0805, update silkscreen
Parts:
- C1, C4: footprint Capacitor_SMD:C_0402_1005Metric -> Capacitor_SMD:C_0805_2012Metric
Changed lines of the file:
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@@
 			)
 		)
-		(property "Footprint" "Capacitor_SMD:C_0402_1005Metric"
+		(property "Footprint" "Capacitor_SMD:C_0805_2012Metric"
 			(at 99.06 43.18 0)
 			(effects
@@
 			)
 		)
-		(property "Footprint" "Capacitor_SMD:C_0402_1005Metric"
+		(property "Footprint" "Capacitor_SMD:C_0805_2012Metric"
 			(at 124.46 43.18 0)
 			(effects
